File: hardware/imu-v3.kicad_pcb (KiCad board)
At the start: 2 copper layers, 25 x 25 mm, 32 parts, among them P1 CON-SENSOR2, P2 BOOT, P3 DEBUG, U1 XMC1302, U2 BNO055, U3 DRILL, U4 DRILL, U5 DRILL, U6 DRILL, X1 32.768kHz

Commit message: ready for prototype
Parts:
- U1: value XMC1302 -> XMC1XXX
Connections:
- U1 pad 18: BNO-BOOT -> BNO-ADR-SELECT
- U1 pad 19: BNO-ADR-SELECT -> BNO-INT
- U1 pad 20: BNO-INT -> BNO-nRESET
- U1 pad 21: BNO-nRESET -> BNO-BOOT
Routing:
- net BNO-BOOT: track 12.6 -> 16.1 mm, vias 2 -> 0
- net GND: track 36.2 -> 33.4 mm, vias 26 -> 28

Commit message: changed silkscreen
Parts:
- moved G*** 9.48 mm to (169.9, 69.2), turned to 90 degrees
- moved VAL 8.77 mm to (170.0, 56.3), turned to 90 degrees
- turned VAL to 90 degrees
Changed lines of the file:
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@@
   )
   (setup
-    (last_trace_width 0.2)
+    (last_trace_width 0.15)
     (user_trace_width 0.15)
     (user_trace_width 0.2)
@@
   )
   (module kicad-libraries:WEEE_7mm (layer B.Cu)
-    (at 163.8 62.5 180)
-    (fp_text reference VAL (at 0 0) (layer B.SilkS) hide
+    (at 170 56.3 90)
+    (fp_text reference VAL (at 0 0 90) (layer B.SilkS) hide
       (effects (font (size 0.2 0.2) (thickness 0.05)) (justify mirror))
     )
-    (fp_text value WEEE_7mm (at 0.75 0) (layer B.SilkS) hide
+    (fp_text value WEEE_7mm (at 0.75 0 90) (layer B.SilkS) hide
       (effects (font (size 0.2 0.2) (thickness 0.05)) (justify mirror))
     )
@@
   )
   (module kicad-libraries:Logo_CoMCU (layer B.Cu)
-    (at 176.7 62.6 180)
-    (fp_text reference G*** (at 0 0) (layer B.SilkS) hide
+    (at 169.9 69.2 90)
+    (fp_text reference G*** (at 0 0 90) (layer B.SilkS) hide
       (effects (font (size 1.524 1.524) (thickness 0.3)) (justify mirror))
     )
-    (fp_text value LOGO (at 0.75 0) (layer B.SilkS) hide
+    (fp_text value LOGO (at 0.75 0 90) (layer B.SilkS) hide
       (effects (font (size 1.524 1.524) (thickness 0.3)) (justify mirror))
     )
@@
   )
   (module kicad-libraries:CE_5mm (layer B.Cu)
-    (at 170 62.5 180)
-    (fp_text reference VAL (at 0 0) (layer B.SilkS) hide
+    (at 170 62.5 90)
+    (fp_text reference VAL (at 0 0 90) (layer B.SilkS) hide
       (effects (font (size 0.2 0.2) (thickness 0.05)) (justify mirror))
     )
-    (fp_text value CE_5mm (at 0 0) (layer B.SilkS) hide
+    (fp_text value CE_5mm (at 0 0 90) (layer B.SilkS) hide
       (effects (font (size 0.2 0.2) (thickness 0.05)) (justify mirror))
     )
@@
   )
   (zone (net 1) (net_name GND) (layer F.Cu) (hatch edge 0.508)
-    (connect_pads yes (clearance 0.508))
+    (connect_pads yes (clearance 0.15))
     (min_thickness 0.254)
     (fill yes (arc_segments 32) (thermal_gap 0.508) (thermal_bridge_width 0.508))
