File: hardware/imu-v3.kicad_pcb (KiCad board)
At the start: 2 copper layers, 25 x 25 mm, 32 parts, among them P1 CON-SENSOR2, P2 BOOT, P3 DEBUG, U1 XMC1XXX, U2 BNO055, U3 DRILL, U4 DRILL, U5 DRILL, U6 DRILL, X1 32.768kHz

Commit message: specify processor as XMC1302
Parts:
- U1: value XMC1XXX -> XMC1302
